File: UINIO-Keyboard.kicad_sch (KiCad schematic)
At the start: 0 parts

Commit message: Update
Parts:
- added R1, R2, R3, R4, R5, R6, R7, R8: 10K, symbol Device:R
- added SW1, SW10, SW11, SW12, SW13, SW14, SW15, SW16, SW17, SW18, SW19, SW2, SW20, SW21, SW22, SW23, SW24, SW25, SW26, SW27, SW28, SW29, SW3, SW30, SW31, SW32, SW33, SW34, SW35, SW36, SW37, SW38, SW39, SW4, SW40, SW41, SW42, SW43, SW44, SW45, SW46, SW47, SW48, SW49, SW5, SW50, SW51, SW52, SW53, SW54, SW55, SW56, SW57, SW58, SW59, SW6, SW60, SW61, SW62, SW63, SW64, SW7, SW8, SW9: A, Uinio:KEY-SMD_4P-L4.2-W3.4-P2.15-LS4.7, symbol Uinio:Key_YTS_A016S_1
- added U1: CH452A, Uinio:SOIC-28_L17.9-W7.5-P1.27-LS10.3-BL, symbol Uinio:CH452A
Connections:
- new net: R4.2, SW13.1, SW13.2, SW21.1, SW21.2, SW29.1, SW29.2, SW37.1, SW37.2, SW45.1, SW45.2, SW5.1, SW5.2, SW53.1, SW53.2, SW61.1, SW61.2
- new net: R1.2, SW16.1, SW16.2, SW24.1, SW24.2, SW32.1, SW32.2, SW40.1, SW40.2, SW48.1, SW48.2, SW56.1, SW56.2, SW64.1, SW64.2, SW8.1, SW8.2
- new net: R3.2, SW14.1, SW14.2, SW22.1, SW22.2, SW30.1, SW30.2, SW38.1, SW38.2, SW46.1, SW46.2, SW54.1, SW54.2, SW6.1, SW6.2, SW62.1, SW62.2
- new net: R6.2, SW11.1, SW11.2, SW19.1, SW19.2, SW27.1, SW27.2, SW3.1, SW3.2, SW35.1, SW35.2, SW43.1, SW43.2, SW51.1, SW51.2, SW59.1, SW59.2
- new net: R5.2, SW12.1, SW12.2, SW20.1, SW20.2, SW28.1, SW28.2, SW36.1, SW36.2, SW4.1, SW4.2, SW44.1, SW44.2, SW52.1, SW52.2, SW60.1, SW60.2
- new net: R2.2, SW15.1, SW15.2, SW23.1, SW23.2, SW31.1, SW31.2, SW39.1, SW39.2, SW47.1, SW47.2, SW55.1, SW55.2, SW63.1, SW63.2, SW7.1, SW7.2
- new net: R8.2, SW1.1, SW1.2, SW17.1, SW17.2, SW25.1, SW25.2, SW33.1, SW33.2, SW41.1, SW41.2, SW49.1, SW49.2, SW57.1, SW57.2, SW9.1, SW9.2
- new net: R7.2, SW10.1, SW10.2, SW18.1, SW18.2, SW2.1, SW2.2, SW26.1, SW26.2, SW34.1, SW34.2, SW42.1, SW42.2, SW50.1, SW50.2, SW58.1, SW58.2
- new net DCLK: U1.27 (DCLK)
- new net DIG0: R1.1, U1.8 (DIG0)
- new net DIG1: R2.1, U1.7 (DIG1)
- new net DIG2: R3.1, U1.6 (DIG2)
- new net DIG3: R4.1, U1.5 (DIG3)
- new net DIG4: R5.1, U1.4 (DIG4)
- new net DIG5: R6.1, U1.3 (DIG5)
- new net DIG6: R7.1, U1.2 (DIG6)
- new net DIG7: R8.1, U1.1 (DIG7)
- new net DIN: U1.26 (DIN)
- new net DOUT: U1.24 (DOUT)
- new net GND: U1.10 (GND), U1.9 (GND)
- new net H3L2: U1.14 (H3L2)
- new net LOAD: U1.25 (LOAD)
- new net RST: U1.12 (RST)
- new net RST#: U1.13 (RST#)
- new net RSTI: U1.28 (RSTI)
- new net SEG0: SW1.3, SW1.4, SW2.3, SW2.4, SW3.3, SW3.4, SW4.3, SW4.4, SW5.3, SW5.4, SW6.3, SW6.4, SW7.3, SW7.4, SW8.3, SW8.4, U1.15 (SEG0)
- new net SEG1: SW10.3, SW10.4, SW11.3, SW11.4, SW12.3, SW12.4, SW13.3, SW13.4, SW14.3, SW14.4, SW15.3, SW15.4, SW16.3, SW16.4, SW9.3, SW9.4, U1.16 (SEG1)
- new net SEG2: SW17.3, SW17.4, SW18.3, SW18.4, SW19.3, SW19.4, SW20.3, SW20.4, SW21.3, SW21.4, SW22.3, SW22.4, SW23.3, SW23.4, SW24.3, SW24.4, U1.17 (SEG2)
- new net SEG3: SW25.3, SW25.4, SW26.3, SW26.4, SW27.3, SW27.4, SW28.3, SW28.4, SW29.3, SW29.4, SW30.3, SW30.4, SW31.3, SW31.4, SW32.3, SW32.4, U1.18 (SEG3)
- new net SEG4: SW33.3, SW33.4, SW34.3, SW34.4, SW35.3, SW35.4, SW36.3, SW36.4, SW37.3, SW37.4, SW38.3, SW38.4, SW39.3, SW39.4, SW40.3, SW40.4, U1.19 (SEG4)
- new net SEG5: SW41.3, SW41.4, SW42.3, SW42.4, SW43.3, SW43.4, SW44.3, SW44.4, SW45.3, SW45.4, SW46.3, SW46.4, SW47.3, SW47.4, SW48.3, SW48.4, U1.20 (SEG5)
- new net SEG6: SW49.3, SW49.4, SW50.3, SW50.4, SW51.3, SW51.4, SW52.3, SW52.4, SW53.3, SW53.4, SW54.3, SW54.4, SW55.3, SW55.4, SW56.3, SW56.4, U1.21 (SEG6)
- new net SEG7: SW57.3, SW57.4, SW58.3, SW58.4, SW59.3, SW59.4, SW60.3, SW60.4, SW61.3, SW61.4, SW62.3, SW62.4, SW63.3, SW63.4, SW64.3, SW64.4, U1.22 (SEG7)
- new net VCC: U1.23 (VCC)
- no-connect marks 0 -> 1

Commit message: Update PCB.
Parts:
- added U2, U3, U4: EC1106S, Uinio:SW-SMD_EC1106S, symbol Uinio:EC1106S
- R1, R2, R3, R4, R5, R6, R7, R8: footprint (none) -> Resistor_SMD:R_0603_1608Metric
Changed lines of the file:
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@@
       (effects (font (size 1.27 1.27)) (justify left))
     )
-    (property "Footprint" "" (at 194.31 240.538 90)
+    (property "Footprint" "Resistor_SMD:R_0603_1608Metric" (at 194.31 240.538 90)
       (effects (font (size 1.27 1.27)) hide)
     )
@@
       (effects (font (size 1.27 1.27)) (justify left))
     )
-    (property "Footprint" "" (at 194.31 255.778 90)
+    (property "Footprint" "Resistor_SMD:R_0603_1608Metric" (at 194.31 255.778 90)
       (effects (font (size 1.27 1.27)) hide)
     )
@@
       (effects (font (size 1.27 1.27)) (justify left))
     )
-    (property "Footprint" "" (at 194.31 235.458 90)
+    (property "Footprint" "Resistor_SMD:R_0603_1608Metric" (at 194.31 235.458 90)
       (effects (font (size 1.27 1.27)) hide)
     )
@@
         (path "/bbcda099-2b9a-49b2-9355-114c31909b50"
           (reference "SW47") (unit 1)
+        )
+      )
+    )
+  )
+  (symbol (lib_id "Uinio:EC1106S") (at 322.58 134.62 0) (unit 1)
+    (in_bom yes) (on_board yes) (dnp no)
+    (property "Reference" "U3" (at 322.58 121.92 0)
+      (effects (font (size 1.27 1.27)))
+    )
+    (property "Value" "EC1106S" (at 322.58 148.59 0)
+      (effects (font (size 1.27 1.27)))
+    )
+    (property "Footprint" "Uinio:SW-SMD_EC1106S" (at 323.85 148.59 0)
+      (effects (font (size 1.27 1.27)) hide)
+    )
+    (property "Datasheet" "" (at 322.58 133.0706 0)
+      (effects (font (size 1.27 1.27)) hide)
+    )
+    (property "SuppliersPartNumber" "C9900001788" (at 322.58 138.1506 0)
+      (effects (font (size 1.27 1.27)) hide)
+    )
+    (property "uuid" "std:9323c30b97424b91b0b9012d0e3352f8" (at 322.58 138.1506 0)
+      (effects (font (size 1.27 1.27)) hide)
+    )
+    (pin "1")
+    (pin "2")
+    (pin "3")
+    (pin "4")
+    (pin "5")
+    (pin "6")
+    (pin "7")
+    (instances
+      (project "UINIO-Keyboard"
+        (path "/bbcda099-2b9a-49b2-9355-114c31909b50"
+          (reference "U3") (unit 1)
         )
       )
@@
       (effects (font (size 1.27 1.27)) (justify left))
     )
-    (property "Footprint" "" (at 194.31 260.858 90)
+    (property "Footprint" "Resistor_SMD:R_0603_1608Metric" (at 194.31 260.858 90)
       (effects (font (size 1.27 1.27)) hide)
     )
@@
       (effects (font (size 1.27 1.27)) (justify left))
     )
-    (property "Footprint" "" (at 194.31 265.938 90)
+    (property "Footprint" "Resistor_SMD:R_0603_1608Metric" (at 194.31 265.938 90)
       (effects (font (size 1.27 1.27)) hide)
     )
@@
       (effects (font (size 1.27 1.27)) (justify left))
     )
-    (property "Footprint" "" (at 194.31 271.018 90)
+    (property "Footprint" "Resistor_SMD:R_0603_1608Metric" (at 194.31 271.018 90)
       (effects (font (size 1.27 1.27)) hide)
     )
@@
         (path "/bbcda099-2b9a-49b2-9355-114c31909b50"
           (reference "R8") (unit 1)
+        )
+      )
+    )
+  )
+  (symbol (lib_id "Uinio:EC1106S") (at 350.52 134.62 0) (unit 1)
+    (in_bom yes) (on_board yes) (dnp no)
+    (property "Reference" "U4" (at 350.52 121.92 0)
+      (effects (font (size 1.27 1.27)))
+    )
+    (property "Value" "EC1106S" (at 350.52 148.59 0)
+      (effects (font (size 1.27 1.27)))
+    )
+    (property "Footprint" "Uinio:SW-SMD_EC1106S" (at 351.79 148.59 0)
+      (effects (font (size 1.27 1.27)) hide)
+    )
+    (property "Datasheet" "" (at 350.52 133.0706 0)
+      (effects (font (size 1.27 1.27)) hide)
+    )
+    (property "SuppliersPartNumber" "C9900001788" (at 350.52 138.1506 0)
+      (effects (font (size 1.27 1.27)) hide)
+    )
+    (property "uuid" "std:9323c30b97424b91b0b9012d0e3352f8" (at 350.52 138.1506 0)
+      (effects (font (size 1.27 1.27)) hide)
+    )
+    (pin "1")
+    (pin "2")
+    (pin "3")
+    (pin "4")
+    (pin "5")
+    (pin "6")
+    (pin "7")
+    (instances
+      (project "UINIO-Keyboard"
+        (path "/bbcda099-2b9a-49b2-9355-114c31909b50"
+          (reference "U4") (unit 1)
         )
       )
@@
       (effects (font (size 1.27 1.27)) (justify left))
     )
-    (property "Footprint" "" (at 194.31 250.698 90)
+    (property "Footprint" "Resistor_SMD:R_0603_1608Metric" (at 194.31 250.698 90)
       (effects (font (size 1.27 1.27)) hide)
     )
@@
         (path "/bbcda099-2b9a-49b2-9355-114c31909b50"
           (reference "SW63") (unit 1)
+        )
+      )
+    )
+  )
+  (symbol (lib_id "Uinio:EC1106S") (at 294.64 134.62 0) (unit 1)
+    (in_bom yes) (on_board yes) (dnp no)
+    (property "Reference" "U2" (at 294.64 121.92 0)
+      (effects (font (size 1.27 1.27)))
+    )
+    (property "Value" "EC1106S" (at 294.64 148.59 0)
+      (effects (font (size 1.27 1.27)))
+    )
+    (property "Footprint" "Uinio:SW-SMD_EC1106S" (at 295.91 148.59 0)
+      (effects (font (size 1.27 1.27)) hide)
+    )
+    (property "Datasheet" "" (at 294.64 133.0706 0)
+      (effects (font (size 1.27 1.27)) hide)
+    )
+    (property "SuppliersPartNumber" "C9900001788" (at 294.64 138.1506 0)
+      (effects (font (size 1.27 1.27)) hide)
+    )
+    (property "uuid" "std:9323c30b97424b91b0b9012d0e3352f8" (at 294.64 138.1506 0)
+      (effects (font (size 1.27 1.27)) hide)
+    )
+    (pin "1")
+    (pin "2")
+    (pin "3")
+    (pin "4")
+    (pin "5")
+    (pin "6")
+    (pin "7")
+    (instances
+      (project "UINIO-Keyboard"
+        (path "/bbcda099-2b9a-49b2-9355-114c31909b50"
+          (reference "U2") (unit 1)
         )
       )
@@
       (effects (font (size 1.27 1.27)) (justify left))
     )
-    (property "Footprint" "" (at 194.31 245.618 90)
-      (effects (font (size 1.27 1.27)) hide)
-    )
+    (property "Footprint" "Resistor_SMD:R_0603_1608Metric" (at 194.31 245.618 90)
+      (effects (font (size 1.27 1.27)) hide)
+    )

Commit message: update
Parts:
- added C1: 0.1uF, symbol Device:C
- added J1: Conn_01x06_Pin, symbol Connector:Conn_01x06_Pin
- added R9: 10K, symbol Device:R
Connections:
- net DIN is gone; now on net GND: U1.26 (DIN)
- net DCLK: now also J1.6 (Pin_6)
- net DOUT: now also J1.2 (Pin_2)
- net GND: now also U2.5 (D), U2.6 (EP), U2.7 (EP), C1.2, J1.4 (Pin_4), J1.5 (Pin_5)
- net RST#: now also J1.1 (Pin_1)
- net VCC: now also C1.1, J1.3 (Pin_3)
- net at U2.4 (E): now also R9.1
Other:
- moved on the sheet: U1, U2, U3, U4

Commit message: Complete schematic drawing.
Parts:
- removed U4: EC1106S, Uinio:SW-SMD_EC1106S, symbol Uinio:EC1106S
- added C1, C2, C3, C4, C5, C6: 0.01uF, Capacitor_SMD:C_0402_1005Metric, symbol Device:C
- added D1: LED_Red, LED_SMD:LED_0603_1608Metric, symbol Device:LED
- added J2, J3: Conn_01x05_Pin, Connector_PinHeader_2.54mm:PinHeader_1x05_P2.54mm_Vertical, symbol Connector:Conn_01x05_Pin
- added R10, R11, R12, R13, R14: 10K, Resistor_SMD:R_0402_1005Metric, symbol Device:R
- added R3: 2K, Resistor_SMD:R_0402_1005Metric, symbol Device:R
- C7: renamed from C1; footprint (none) -> Capacitor_SMD:C_0402_1005Metric
- J1: footprint (none) -> Connector_PinHeader_2.54mm:PinHeader_1x06_P2.54mm_Vertical
- R1, R2, R3, R4, R5, R6, R7, R8: footprint Resistor_SMD:R_0603_1608Metric -> Resistor_SMD:R_0402_1005Metric
- R9: footprint (none) -> Resistor_SMD:R_0402_1005Metric
- renumbered SW1 to K1, SW10 to K10, SW18 to K11, SW26 to K12, SW34 to K13, SW42 to K14, SW50 to K15, SW58 to K16, SW3 to K17, SW11 to K18, SW19 to K19, SW9 to K2, SW27 to K20, SW35 to K21, SW43 to K22, SW51 to K23, SW59 to K24, SW4 to K25, SW12 to K26, SW20 to K27, SW28 to K28, SW36 to K29, SW17 to K3, SW44 to K30, SW52 to K31, SW60 to K32, SW5 to K33, SW13 to K34, SW21 to K35, SW29 to K36, SW37 to K37, SW45 to K38, SW53 to K39, SW25 to K4, SW61 to K40, SW6 to K41, SW14 to K42, SW22 to K43, SW30 to K44, SW38 to K45, SW46 to K46, SW54 to K47, SW62 to K48, SW7 to K49, SW33 to K5, SW15 to K50, SW23 to K51, SW31 to K52, SW39 to K53, SW47 to K54, SW55 to K55, SW63 to K56, SW8 to K57, SW16 to K58, SW24 to K59, SW41 to K6, SW32 to K60, SW40 to K61, SW48 to K62, SW56 to K63, SW64 to K64, SW49 to K7, SW57 to K8, SW2 to K9
Connections:
- net H3L2 is gone; now on net GND: U1.14 (H3L2)
- net VCC is gone; now on net LOAD: C7.1, J1.3 (Pin_3), U1.23 (VCC)
- net GND: now also D1.1 (K); no longer U2.5 (D), U2.6 (EP), U2.7 (EP)
- net LOAD: now also R3.2
- net EC11-A-2: now reaches U3.1 (A)
- net EC11-A-2: now also C2.1, J3.5 (Pin_5), R12.1
- net EC11-GND-2: now reaches U3.2 (C)
- net EC11-GND-2: now also U3.4 (E), U3.6 (EP), U3.7 (EP), C2.2, C4.2, C6.2, J3.2 (Pin_2)
- net EC11-B-2: now reaches U3.3 (B)
- net EC11-B-2: now also C6.1, J3.4 (Pin_4), R14.1
- net EC11-E-2: now reaches U3.5 (D)
- net EC11-E-2: now also C4.1, J3.3 (Pin_3), R11.1
- net EC11-A-1: now reaches U2.1 (A)
- net EC11-A-1: now also C1.1, J2.5 (Pin_5), R10.1
- net EC11-GND-1: now reaches U2.2 (C)
- net EC11-GND-1: now also U2.4 (E), U2.6 (EP), U2.7 (EP), C1.2, C3.2, C5.2, J2.2 (Pin_2)
- net EC11-B-1: now reaches U2.3 (B)
- net EC11-B-1: now also C5.1, J2.4 (Pin_4), R13.1
- net EC11-E-1: now reaches R9.1
- net EC11-E-1: now also U2.5 (D), C3.1, J2.3 (Pin_3); no longer U2.4 (E)
- net EC11-VCC-1: now reaches R9.2
- net EC11-VCC-1: now also J2.1 (Pin_1), R10.2, R13.2
- net RST: no longer names the net of U1.12 (RST)
- net RSTI: no longer names the net of U1.28 (RSTI)
- new net: D1.2 (A), R3.1
- new net EC11-VCC-2: J3.1 (Pin_1), R11.2, R12.2, R14.2
- no-connect marks 1 -> 3
Other:
- moved on the sheet: C7, J1, K1, K10, K11, K12, K13, K14, K15, K16, K17, K18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

Commit message: PCB Layout.
Parts:
- added D1 (x2): LED_Red, LED_SMD:LED_0603_1608Metric, symbol Device:LED
- added J4: Conn_01x05_Pin, Connector_PinHeader_2.54mm:PinHeader_1x05_P2.54mm_Vertical, symbol Connector:Conn_01x05_Pin
- added R3 (x2): 2K, Resistor_SMD:R_0402_1005Metric, symbol Device:R
- added SW2: RKJXV1224005, Uinio:SW-TH_RKJXV1224005, symbol Uinio:RKJXV1224005
Connections:
- net EC11-VCC-1: now also R3.2
- net EC11-VCC-2: now also R3.2
- net GND: now also D1.1 (K), D1.1 (K)
- new net: D1.2 (A), R3.1 (x2)
- new net: SW2.a, SW2.b
- new net: SW2.c, SW2.d
Other:
- note added: "8 * 8 矩阵键盘"
- note added: "EC11 旋转编码器"
- note added: "RKJXV 模拟量摇杆"
- moved on the sheet: C1, C2, C3, C4, C5, C6, C7, D1, J1, J2, J3, R10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

Commit message: Update PCB.
Connections:
- net at SW2.10 (GND): now also SW2.9 (GND)
- net at SW2.7 (GND): now also SW2.8 (GND)
- net at SW2.a: now also SW2.c; no longer SW2.b
- net at SW2.d: now also SW2.b; no longer SW2.c
Changed lines of the file:
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@@
+    (stroke (width 0) (type default))
+  )
+  (wire (pts (xy 305.435 283.21) (xy 305.435 298.45))
     (stroke (width 0) (type default))
   )
@@
     (stroke (width 0) (type default))
   )
+  (wire (pts (xy 316.23 298.45) (xy 316.865 298.45))
+    (stroke (width 0) (type default))
+  )
   (wire (pts (xy 86.36 118.11) (xy 81.28 118.11))
     (stroke (width 0) (type default))
@@
     (stroke (width 0) (type default))
   )
+  (wire (pts (xy 318.77 285.75) (xy 318.77 295.91))
+    (stroke (width 0) (type default))
+  )
   (wire (pts (xy 132.08 144.78) (xy 127 144.78))
     (stroke (width 0) (type default))
@@
     (stroke (width 0) (type default))
   )
+  (wire (pts (xy 339.09 285.75) (xy 360.045 285.75))
+    (stroke (width 0) (type default))
+  )
   (wire (pts (xy 96.52 40.64) (xy 91.44 40.64))
     (stroke (width 0) (type default))
@@
     (stroke (width 0) (type default))
   )
+  (wire (pts (xy 360.045 285.75) (xy 360.045 295.91))
+    (stroke (width 0) (type default))
+  )
   (wire (pts (xy 149.86 210.82) (xy 149.86 220.98))
     (stroke (width 0) (type default))
@@
     (stroke (width 0) (type default))
   )
+  (wire (pts (xy 316.865 298.45) (xy 316.865 283.21))
+    (stroke (width 0) (type default))
+  )
   (wire (pts (xy 187.96 81.28) (xy 187.96 91.44))
     (stroke (width 0) (type default))
@@
     (stroke (width 0) (type default))
   )
-  (wire (pts (xy 306.07 298.45) (xy 316.23 298.45))
+  (wire (pts (xy 306.07 283.21) (xy 305.435 283.21))
     (stroke (width 0) (type default))
   )
@@
     (stroke (width 0) (type default))
   )
+  (wire (pts (xy 360.045 295.91) (xy 339.09 295.91))
+    (stroke (width 0) (type default))
+  )
   (wire (pts (xy 96.52 173.99) (xy 73.66 173.99))
     (stroke (width 0) (type default))
@@
     (stroke (width 0) (type default))
   )
+  (wire (pts (xy 305.435 298.45) (xy 306.07 298.45))
+    (stroke (width 0) (type default))
+  )
   (wire (pts (xy 195.58 269.24) (xy 35.56 269.24))
     (stroke (width 0) (type default))
@@
     (stroke (width 0) (type default))
   )
-  (wire (pts (xy 306.07 283.21) (xy 316.23 283.21))
-    (stroke (width 0) (type default))
-  )
   (wire (pts (xy 63.5 54.61) (xy 58.42 54.61))
     (stroke (width 0) (type default))
@@
     (stroke (width 0) (type default))
   )
+  (wire (pts (xy 316.865 283.21) (xy 316.23 283.21))
+    (stroke (width 0) (type default))
+  )

Commit message: Update PCB Layout.
Parts:
- added C10, C8, C9: 0.01uF, Capacitor_SMD:C_0402_1005Metric, symbol Device:C
- added D1 (x2): LED_Red, LED_SMD:LED_0603_1608Metric, symbol Device:LED
- added J5: Conn_01x05_Pin, Connector_PinHeader_2.54mm:PinHeader_1x05_P2.54mm_Vertical, symbol Connector:Conn_01x05_Pin
- added R19, R20, R21: 10K, Resistor_SMD:R_0402_1005Metric, symbol Device:R
- added R3 (x2): 2K, Resistor_SMD:R_0402_1005Metric, symbol Device:R
- added SW1: SWITCH_SS12D00G3, Uinio:SW-TH_SS-12D01-GX, symbol Uinio:SWITCH_SS12D00G3
- added U4: EC1106S, Uinio:SW-SMD_EC1106S, symbol Uinio:EC1106S
Connections:
- net EC11-GND-1: now also D1.1 (K)
- net EC11-GND-2: now also D1.1 (K)
- net GND: no longer D1.1 (K), D1.1 (K)
- net Rocker_GND: now reaches J4.1 (Pin_1)
- net Rocker_GND: now also SW2.3 (A), SW2.6 (B), SW2.a, SW2.c, D1.1 (K), R3.2
- net Rocker_VCC: now reaches J4.2 (Pin_2)
- net Rocker_VCC: now also SW2.1 (B), SW2.4 (A)
- net Rocker_X: now reaches J4.3 (Pin_3)
- net Rocker_X: now also SW2.5 (DTA)
- net Rocker_Y: now reaches J4.4 (Pin_4)
- net Rocker_Y: now also SW2.2 (DTA)
- net Rocker_SW: now reaches J4.5 (Pin_5)
- net Rocker_SW: now also SW2.b, SW2.d
- new net: D1.2 (A), R3.1 (x2)
- new net EC11-A-3: C8.1, J5.5 (Pin_5), R20.1, U4.1 (A)
- new net EC11-B-3: C10.1, J5.4 (Pin_4), R21.1, U4.3 (B)
- new net EC11-E-3: C9.1, J5.3 (Pin_3), R19.1, U4.5 (D)
- new net EC11-GND-3: C10.2, C8.2, C9.2, D1.1 (K), J5.2 (Pin_2), U4.2 (C), U4.4 (E), U4.6 (EP), U4.7 (EP)
- new net EC11-VCC-3: J5.1 (Pin_1), R19.2, R20.2, R21.2, R3.2
Other:
- moved on the sheet: C1, C2, C3, C4, C5, C6, D1, J2, J3, J4, R10, R11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

Commit message: update
Connections:
- net GND: now also SW1.1
- net LOAD: now also SW1.2; no longer C7.1, J1.3 (Pin_3), R3.2, U1.23 (VCC)
- net Rocker_GND: now also J4.5 (Pin_5); no longer J4.1 (Pin_1), R3.2
- net Rocker_SW: now also J4.1 (Pin_1), R3.2; no longer J4.5 (Pin_5)
- net Rocker_VCC: now also J4.4 (Pin_4); no longer J4.2 (Pin_2)
- net Rocker_X: now also J4.2 (Pin_2); no longer J4.3 (Pin_3)
- net Rocker_Y: now also J4.3 (Pin_3); no longer J4.4 (Pin_4)
- net VCC: now reaches SW1.3
- net VCC: now also C7.1, J1.3 (Pin_3), R3.2, U1.23 (VCC)
Other:
- moved on the sheet: C7, D1, J1, R3, SW1, U1
