File: UINIO-Keyboard.kicad_sch (KiCad schematic)
At the start: 112 parts, among them J1 Conn_01x06_Pin, J2 Conn_01x05_Pin, J3 Conn_01x05_Pin, J4 Conn_01x05_Pin, J5 Conn_01x05_Pin, K1 A, K10 A, K11 A, K12 A, K13 A, K14 A, K15 A, K16 A, K17 A, K18 A, K19 A, K2 A, K20 A, K21 A, K22 A, K23 A, K24 A, K25 A, K26 A, K27 A, K28 A, K29 A, K3 A, K30 A, K31 A, K32 A, K33 A, K34 A, K35 A, K36 A, K37 A, K38 A, K39 A, K4 A, K40 A, K41 A, K42 A, K43 A, K44 A, K45 A, K46 A, K47 A, K48 A, K49 A, K5 A, K50 A, K51 A, K52 A, K53 A, K54 A, K55 A, K56 A, K57 A, K58 A, K59 A, K6 A, K60 A, K61 A, K62 A, K63 A, K64 A, K7 A, K8 A, K9 A, SW1 SWITCH_SS12D00G3, SW2 RKJXV1224005, U1 CH452A, U2 EC1106S, U3 EC1106S, U4 EC1106S

Commit message: Complete PCB layout.
Connections:
- net DCLK: now also J1.1 (Pin_1); no longer J1.6 (Pin_6)
- net DOUT: now also J1.3 (Pin_3); no longer J1.2 (Pin_2)
- net GND: now also J1.2 (Pin_2); no longer J1.4 (Pin_4)
- net RST#: now also J1.4 (Pin_4); no longer J1.1 (Pin_1)
- net VCC: now also J1.6 (Pin_6); no longer J1.3 (Pin_3)
Changed lines of the file:
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@@
     (stroke (width 0) (type default))
   )
-  (wire (pts (xy 58.42 323.85) (xy 80.01 323.85))
+  (wire (pts (xy 58.42 326.39) (xy 79.375 326.39))
     (stroke (width 0) (type default))
   )
@@
     (stroke (width 0) (type default))
   )
-  (wire (pts (xy 58.42 328.93) (xy 73.66 328.93))
+  (wire (pts (xy 58.42 316.23) (xy 73.66 316.23))
     (stroke (width 0) (type default))
   )
@@
     (stroke (width 0) (type default))
   )
-  (wire (pts (xy 58.42 326.39) (xy 73.66 326.39))
+  (wire (pts (xy 58.42 318.77) (xy 73.66 318.77))
     (stroke (width 0) (type default))
   )
@@
     (stroke (width 0) (type default))
   )
-  (wire (pts (xy 58.42 321.31) (xy 81.28 321.31))
+  (wire (pts (xy 58.42 328.93) (xy 88.265 328.93))
     (stroke (width 0) (type default))
   )
@@
     (stroke (width 0) (type default))
   )
-  (wire (pts (xy 58.42 318.77) (xy 73.66 318.77))
+  (wire (pts (xy 58.42 321.31) (xy 73.66 321.31))
     (stroke (width 0) (type default))
   )
@@
     (stroke (width 0) (type default))
   )
-  (wire (pts (xy 58.42 316.23) (xy 73.66 316.23))
+  (wire (pts (xy 58.42 323.85) (xy 73.66 323.85))
     (stroke (width 0) (type default))
   )
@@
     (effects (font (size 8 8)) (justify left bottom))
   )
-  (text "8 * 8 矩阵键盘" (at 80.01 364.49 0)
+  (text "8 * 8 矩阵键盘" (at 82.55 374.015 0)
     (effects (font (size 8 8)) (justify left bottom))
   )
@@
     (effects (font (size 1.27 1.27)) (justify left bottom))
   )
-  (label "SCL" (at 63.5 328.93 0) (fields_autoplaced)
+  (label "SCL" (at 63.5 316.23 0) (fields_autoplaced)
     (effects (font (size 1.27 1.27)) (justify left bottom))
   )
@@
     (effects (font (size 1.27 1.27)) (justify right bottom))
   )
-  (label "DOUT" (at 73.66 318.77 0) (fields_autoplaced)
+  (label "DOUT" (at 73.66 321.31 0) (fields_autoplaced)
     (effects (font (size 1.27 1.27)) (justify left bottom))
   )
@@
     (effects (font (size 1.27 1.27)) (justify left bottom))
   )
-  (label "SDA" (at 63.5 326.39 0) (fields_autoplaced)
+  (label "SDA" (at 63.5 318.77 0) (fields_autoplaced)
     (effects (font (size 1.27 1.27)) (justify left bottom))
   )
@@
     (effects (font (size 1.27 1.27)) (justify left bottom))
   )
-  (label "RST#" (at 73.66 316.23 0) (fields_autoplaced)
+  (label "RST#" (at 73.66 323.85 0) (fields_autoplaced)
     (effects (font (size 1.27 1.27)) (justify left bottom))
   )
@@
     (effects (font (size 1.27 1.27)) (justify left bottom))
   )
-  (label "INT#" (at 63.5 318.77 0) (fields_autoplaced)
+  (label "INT#" (at 63.5 321.31 0) (fields_autoplaced)
     (effects (font (size 1.27 1.27)) (justify left bottom))
   )
@@
     (effects (font (size 1.27 1.27)) (justify right bottom))
   )
-  (label "DCLK" (at 73.66 328.93 0) (fields_autoplaced)
+  (label "DCLK" (at 73.66 316.23 0) (fields_autoplaced)
     (effects (font (size 1.27 1.27)) (justify left bottom))
   )
@@
     (effects (font (size 1.27 1.27)) (justify left bottom))
   )
-  (label "VCC" (at 81.28 321.31 0) (fields_autoplaced)
+  (label "VCC" (at 88.265 328.93 0) (fields_autoplaced)
     (effects (font (size 1.27 1.27)) (justify left bottom))
   )
-  (label "DIN" (at 73.66 326.39 0) (fields_autoplaced)
+  (label "DIN" (at 73.66 318.77 0) (fields_autoplaced)
     (effects (font (size 1.27 1.27)) (justify left bottom))
   )
@@
     )
   )
-  (symbol (lib_id "power:GND") (at 80.01 323.85 90) (unit 1)
+  (symbol (lib_id "power:GND") (at 79.375 326.39 90) (mirror x) (unit 1)
     (in_bom yes) (on_board yes) (dnp no)
-    (property "Reference" "#PWR01" (at 86.36 323.85 0)
+    (property "Reference" "#PWR01" (at 85.725 326.39 0)
       (effects (font (size 1.27 1.27)) hide)
     )
-    (property "Value" "GND" (at 82.55 323.85 90)
+    (property "Value" "GND" (at 81.915 326.39 90)
       (effects (font (size 1.27 1.27)) (justify right))
     )
-    (property "Footprint" "" (at 80.01 323.85 0)
+    (property "Footprint" "" (at 79.375 326.39 0)
       (effects (font (size 1.27 1.27)) hide)
     )
-    (property "Datasheet" "" (at 80.01 323.85 0)
+    (property "Datasheet" "" (at 79.375 326.39 0)
       (effects (font (size 1.27 1.27)) hide)
     )

Commit message: Update PCB.
Connections:
- net GND: no longer J1.2 (Pin_2), U1.26 (DIN)
- net RST: now reaches U1.12 (RST)
- net RST: now also J1.4 (Pin_4)
- net EC11-E-1 renamed EC11-D-1
- net EC11-E-2 renamed EC11-D-2
- net EC11-E-3 renamed EC11-D-3
- net RST#: no longer names the net of U1.13 (RST#)
- net RST#: no longer J1.4 (Pin_4)
- new net DIN: J1.2 (Pin_2), U1.26 (DIN)
Changed lines of the file:
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@@
   )
   (no_connect (at 121.92 334.01))
-  (no_connect (at 121.92 336.55))
+  (no_connect (at 121.92 339.09))
   (no_connect (at 162.56 308.61))
   (wire (pts (xy 336.55 76.2) (xy 341.63 76.2))
@@
     (stroke (width 0) (type default))
   )
-  (wire (pts (xy 162.56 313.69) (xy 171.45 313.69))
-    (stroke (width 0) (type default))
-  )
   (wire (pts (xy 40.64 64.77) (xy 35.56 64.77))
     (stroke (width 0) (type default))
@@
     (stroke (width 0) (type default))
   )
-  (wire (pts (xy 120.65 339.09) (xy 121.92 339.09))
-    (stroke (width 0) (type default))
-  )
   (wire (pts (xy 58.42 144.78) (xy 58.42 161.29))
     (stroke (width 0) (type default))
@@
     (stroke (width 0) (type default))
   )
+  (wire (pts (xy 162.56 313.69) (xy 163.83 313.69))
+    (stroke (width 0) (type default))
+  )
   (wire (pts (xy 187.96 196.85) (xy 187.96 199.39))
     (stroke (width 0) (type default))
@@
   )
   (wire (pts (xy 177.8 220.98) (xy 172.72 220.98))
+    (stroke (width 0) (type default))
+  )
+  (wire (pts (xy 119.38 336.55) (xy 121.92 336.55))
     (stroke (width 0) (type default))
   )
@@
     (effects (font (size 1.27 1.27)) (justify left bottom))
   )
-  (label "EC11-E-3" (at 275.59 208.28 0) (fields_autoplaced)
+  (label "EC11-D-3" (at 275.59 208.28 0) (fields_autoplaced)
     (effects (font (size 1.27 1.27)) (justify left bottom))
   )
@@
     (effects (font (size 1.27 1.27)) (justify right bottom))
   )
-  (label "EC11-E-2" (at 316.23 102.87 180) (fields_autoplaced)
+  (label "EC11-D-2" (at 316.23 102.87 180) (fields_autoplaced)
     (effects (font (size 1.27 1.27)) (justify right bottom))
   )
@@
     (effects (font (size 1.27 1.27)) (justify left bottom))
   )
-  (label "EC11-E-2" (at 276.86 137.16 0) (fields_autoplaced)
+  (label "EC11-D-2" (at 276.86 137.16 0) (fields_autoplaced)
     (effects (font (size 1.27 1.27)) (justify left bottom))
   )
@@
     (effects (font (size 1.27 1.27)) (justify left bottom))
   )
-  (label "GND" (at 171.45 313.69 0) (fields_autoplaced)
-    (effects (font (size 1.27 1.27)) (justify left bottom))
-  )
-  (label "RST#" (at 120.65 339.09 180) (fields_autoplaced)
+  (label "RST" (at 119.38 336.55 180) (fields_autoplaced)
     (effects (font (size 1.27 1.27)) (justify right bottom))
   )
@@
     (effects (font (size 1.27 1.27)) (justify left bottom))
   )
-  (label "EC11-E-1" (at 275.59 68.58 0) (fields_autoplaced)
+  (label "EC11-D-1" (at 275.59 68.58 0) (fields_autoplaced)
     (effects (font (size 1.27 1.27)) (justify left bottom))
   )
@@
     (effects (font (size 1.27 1.27)) (justify right bottom))
   )
-  (label "EC11-E-1" (at 316.23 31.75 180) (fields_autoplaced)
+  (label "EC11-D-1" (at 316.23 31.75 180) (fields_autoplaced)
     (effects (font (size 1.27 1.27)) (justify right bottom))
   )
@@
     (effects (font (size 1.27 1.27)) (justify left bottom))
   )
-  (label "RST#" (at 73.66 323.85 0) (fields_autoplaced)
+  (label "RST" (at 73.66 323.85 0) (fields_autoplaced)
     (effects (font (size 1.27 1.27)) (justify left bottom))
   )
@@
     (effects (font (size 1.27 1.27)) (justify left bottom))
   )
-  (label "EC11-E-3" (at 308.61 173.99 180) (fields_autoplaced)
+  (label "EC11-D-3" (at 308.61 173.99 180) (fields_autoplaced)
     (effects (font (size 1.27 1.27)) (justify right bottom))
   )

Commit message: Update PCB.
Parts:
- C3, C4, C9: value 0.01uF -> 0.1uF
Connections:
- net EC11-GND-1 is gone; now on net GND: C1.2, C3.2, C5.2, D1.1 (K), J2.2 (Pin_2), U2.2 (C), U2.4 (E), U2.6 (EP), U2.7 (EP)
- net EC11-GND-2 is gone; now on net GND: C2.2, C4.2, C6.2, D1.1 (K), J3.2 (Pin_2), U3.2 (C), U3.4 (E), U3.6 (EP), U3.7 (EP)
- net EC11-GND-3 is gone; now on net GND: C10.2, C8.2, C9.2, D1.1 (K), J5.2 (Pin_2), U4.2 (C), U4.4 (E), U4.6 (EP), U4.7 (EP)
- net EC11-A-1: now also J2.4 (Pin_4); no longer J2.5 (Pin_5)
- net EC11-A-2: now also J3.4 (Pin_4); no longer J3.5 (Pin_5)
- net EC11-A-3: now also J5.4 (Pin_4); no longer J5.5 (Pin_5)
- net EC11-B-1: now also J2.5 (Pin_5); no longer J2.4 (Pin_4)
- net EC11-B-2: now also J3.5 (Pin_5); no longer J3.4 (Pin_4)
- net EC11-B-3: now also J5.5 (Pin_5); no longer J5.4 (Pin_4)
- net Rocker_GND: now also J4.4 (Pin_4); no longer J4.5 (Pin_5)
- net Rocker_SW: now also J4.3 (Pin_3); no longer J4.1 (Pin_1), R3.2
- net Rocker_VCC: now also J4.5 (Pin_5), R3.2; no longer J4.4 (Pin_4)
- net Rocker_X: now also J4.1 (Pin_1); no longer J4.2 (Pin_2)
- net Rocker_Y: now also J4.2 (Pin_2); no longer J4.3 (Pin_3)
Other:
- moved on the sheet: D1, J4, R3

Commit message: Update PCB.
Connections:
- net Rocker_GND is gone; now on net GND: D1.1 (K), J4.4 (Pin_4), SW2.3 (A), SW2.6 (B), SW2.a, SW2.c
- net GND: now also SW2.10 (GND), SW2.7 (GND), SW2.8 (GND), SW2.9 (GND)
