File: UINIO-Keyboard.kicad_sch (KiCad schematic)
At the start: 112 parts, among them J1 Conn_01x06_Pin, J2 Conn_01x05_Pin, J3 Conn_01x05_Pin, J4 Conn_01x05_Pin, J5 Conn_01x05_Pin, K1 A, K10 A, K11 A, K12 A, K13 A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

Commit message: Release UINIO-Keyboard version 3.1.1.
Other:
- company: 电子技术博客 UinIO.com -> UinIO.com 电子技术实验室
- moved on the sheet: D1, J4, R3
