File: UINIO-Keyboard.kicad_pcb (KiCad board)
At the start: 2 copper layers, 0 parts

Commit message: Complete schematic drawing.
Parts:
- added C1: 0.01uF, Capacitor_SMD:C_0402_1005Metric, F.Cu at (129.1, 59.6)
- added C2: 0.01uF, Capacitor_SMD:C_0402_1005Metric, F.Cu at (129.1, 61.6)
- added C3: 0.01uF, Capacitor_SMD:C_0402_1005Metric, F.Cu at (129.1, 63.6)
- added C4: 0.01uF, Capacitor_SMD:C_0402_1005Metric, F.Cu at (129.1, 65.5)
- added C5: 0.01uF, Capacitor_SMD:C_0402_1005Metric, F.Cu at (129.1, 67.5)
- added C6: 0.01uF, Capacitor_SMD:C_0402_1005Metric, F.Cu at (129.1, 69.5)
- added C7: 0.1uF, Capacitor_SMD:C_0402_1005Metric, F.Cu at (129.1, 71.5)
- added D1: LED_Red, LED_SMD:LED_0603_1608Metric, F.Cu at (132.1, 53.4)
- added J1: Conn_01x06_Pin, Connector_PinHeader_2.54mm:PinHeader_1x06_P2.54mm_Vertical, F.Cu at (141.2, 53.0)
- added J2: Conn_01x05_Pin, Connector_PinHeader_2.54mm:PinHeader_1x05_P2.54mm_Vertical, F.Cu at (175.6, 53.0)
- added J3: Conn_01x05_Pin, Connector_PinHeader_2.54mm:PinHeader_1x05_P2.54mm_Vertical, F.Cu at (109.3, 53.0)
- added K1: A, Uinio:KEY-SMD_4P-L4.2-W3.4-P2.15-LS4.7, F.Cu at (108.8, 78.3)
- added K10: A, Uinio:KEY-SMD_4P-L4.2-W3.4-P2.15-LS4.7, F.Cu at (117.3, 97.8)
- added K11: A, Uinio:KEY-SMD_4P-L4.2-W3.4-P2.15-LS4.7, F.Cu at (126.0, 97.8)
- added K12: A, Uinio:KEY-SMD_4P-L4.2-W3.4-P2.15-LS4.7, F.Cu at (134.6, 97.8)
- added K13: A, Uinio:KEY-SMD_4P-L4.2-W3.4-P2.15-LS4.7, F.Cu at (108.8, 107.6)
- added K14: A, Uinio:KEY-SMD_4P-L4.2-W3.4-P2.15-LS4.7, F.Cu at (117.3, 107.6)
- added K15: A, Uinio:KEY-SMD_4P-L4.2-W3.4-P2.15-LS4.7, F.Cu at (126.0, 107.6)
- added K16: A, Uinio:KEY-SMD_4P-L4.2-W3.4-P2.15-LS4.7, F.Cu at (134.6, 107.6)
- added K17: A, Uinio:KEY-SMD_4P-L4.2-W3.4-P2.15-LS4.7, F.Cu at (108.8, 117.5)
- added K18: A, Uinio:KEY-SMD_4P-L4.2-W3.4-P2.15-LS4.7, F.Cu at (117.3, 117.5)
- added K19: A, Uinio:KEY-SMD_4P-L4.2-W3.4-P2.15-LS4.7, F.Cu at (126.0, 117.5)
- added K2: A, Uinio:KEY-SMD_4P-L4.2-W3.4-P2.15-LS4.7, F.Cu at (117.3, 78.3)
- added K20: A, Uinio:KEY-SMD_4P-L4.2-W3.4-P2.15-LS4.7, F.Cu at (134.6, 117.5)
- added K21: A, Uinio:KEY-SMD_4P-L4.2-W3.4-P2.15-LS4.7, F.Cu at (143.2, 117.5)
- added K22: A, Uinio:KEY-SMD_4P-L4.2-W3.4-P2.15-LS4.7, F.Cu at (151.8, 117.5)
- added K23: A, Uinio:KEY-SMD_4P-L4.2-W3.4-P2.15-LS4.7, F.Cu at (160.4, 117.5)
- added K24: A, Uinio:KEY-SMD_4P-L4.2-W3.4-P2.15-LS4.7, F.Cu at (169.0, 117.5)
- added K25: A, Uinio:KEY-SMD_4P-L4.2-W3.4-P2.15-LS4.7, F.Cu at (177.6, 117.5)
- added K26: A, Uinio:KEY-SMD_4P-L4.2-W3.4-P2.15-LS4.7, F.Cu at (186.2, 117.5)
- added K27: A, Uinio:KEY-SMD_4P-L4.2-W3.4-P2.15-LS4.7, F.Cu at (113.0, 127.2)
- added K28: A, Uinio:KEY-SMD_4P-L4.2-W3.4-P2.15-LS4.7, F.Cu at (121.6, 127.2)
- added K29: A, Uinio:KEY-SMD_4P-L4.2-W3.4-P2.15-LS4.7, F.Cu at (130.2, 127.2)
- added K3: A, Uinio:KEY-SMD_4P-L4.2-W3.4-P2.15-LS4.7, F.Cu at (126.0, 78.3)
- added K30: A, Uinio:KEY-SMD_4P-L4.2-W3.4-P2.15-LS4.7, F.Cu at (138.8, 127.2)
- added K31: A, Uinio:KEY-SMD_4P-L4.2-W3.4-P2.15-LS4.7, F.Cu at (147.4, 127.2)
- added K32: A, Uinio:KEY-SMD_4P-L4.2-W3.4-P2.15-LS4.7, F.Cu at (156.1, 127.2)
- added K33: A, Uinio:KEY-SMD_4P-L4.2-W3.4-P2.15-LS4.7, F.Cu at (164.7, 127.2)
- added K34: A, Uinio:KEY-SMD_4P-L4.2-W3.4-P2.15-LS4.7, F.Cu at (173.3, 127.2)
- added K35: A, Uinio:KEY-SMD_4P-L4.2-W3.4-P2.15-LS4.7, F.Cu at (181.9, 127.2)
- added K36: A, Uinio:KEY-SMD_4P-L4.2-W3.4-P2.15-LS4.7, F.Cu at (121.6, 137.0)
- added K37: A, Uinio:KEY-SMD_4P-L4.2-W3.4-P2.15-LS4.7, F.Cu at (130.2, 137.0)
- added K38: A, Uinio:KEY-SMD_4P-L4.2-W3.4-P2.15-LS4.7, F.Cu at (138.8, 137.0)
- added K39: A, Uinio:KEY-SMD_4P-L4.2-W3.4-P2.15-LS4.7, F.Cu at (147.4, 137.0)
- added K4: A, Uinio:KEY-SMD_4P-L4.2-W3.4-P2.15-LS4.7, F.Cu at (134.6, 78.3)
- added K40: A, Uinio:KEY-SMD_4P-L4.2-W3.4-P2.15-LS4.7, F.Cu at (156.0, 137.0)
- added K41: A, Uinio:KEY-SMD_4P-L4.2-W3.4-P2.15-LS4.7, F.Cu at (164.6, 137.0)
- added K42: A, Uinio:KEY-SMD_4P-L4.2-W3.4-P2.15-LS4.7, F.Cu at (173.2, 137.0)
- added K43: A, Uinio:KEY-SMD_4P-L4.2-W3.4-P2.15-LS4.7, F.Cu at (108.8, 137.0)
- added K44: A, Uinio:KEY-SMD_4P-L4.2-W3.4-P2.15-LS4.7, F.Cu at (108.8, 146.8)
- added K45: A, Uinio:KEY-SMD_4P-L4.2-W3.4-P2.15-LS4.7, F.Cu at (147.4, 146.8)
- added K46: A, Uinio:KEY-SMD_4P-L4.2-W3.4-P2.15-LS4.7, F.Cu at (186.2, 137.0)
- added K47: A, Uinio:KEY-SMD_4P-L4.2-W3.4-P2.15-LS4.7, F.Cu at (186.2, 146.8)
- added K48: A, Uinio:KEY-SMD_4P-L4.2-W3.4-P2.15-LS4.7, F.Cu at (170.7, 93.3)
- added K49: A, Uinio:KEY-SMD_4P-L4.2-W3.4-P2.15-LS4.7, F.Cu at (178.5, 93.3)
- added K5: A, Uinio:KEY-SMD_4P-L4.2-W3.4-P2.15-LS4.7, F.Cu at (108.8, 88.0)
- added K50: A, Uinio:KEY-SMD_4P-L4.2-W3.4-P2.15-LS4.7, F.Cu at (186.3, 93.3)
- added K51: A, Uinio:KEY-SMD_4P-L4.2-W3.4-P2.15-LS4.7, F.Cu at (178.5, 86.7)
- added K52: A, Uinio:KEY-SMD_4P-L4.2-W3.4-P2.15-LS4.7, F.Cu at (178.5, 100.1)
- added K53: A, Uinio:KEY-SMD_4P-L4.2-W3.4-P2.15-LS4.7, F.Cu at (143.2, 78.3)
- added K54: A, Uinio:KEY-SMD_4P-L4.2-W3.4-P2.15-LS4.7, F.Cu at (143.2, 88.0)
- added K55: A, Uinio:KEY-SMD_4P-L4.2-W3.4-P2.15-LS4.7, F.Cu at (143.2, 97.8)
- added K56: A, Uinio:KEY-SMD_4P-L4.2-W3.4-P2.15-LS4.7, F.Cu at (143.2, 107.6)
- added K57: A, Uinio:KEY-SMD_4P-L4.2-W3.4-P2.15-LS4.7, F.Cu at (151.8, 78.3)
- added K58: A, Uinio:KEY-SMD_4P-L4.2-W3.4-P2.15-LS4.7, F.Cu at (151.8, 88.0)
- added K59: A, Uinio:KEY-SMD_4P-L4.2-W3.4-P2.15-LS4.7, F.Cu at (151.8, 97.8)
- added K6: A, Uinio:KEY-SMD_4P-L4.2-W3.4-P2.15-LS4.7, F.Cu at (117.3, 88.0)
- added K60: A, Uinio:KEY-SMD_4P-L4.2-W3.4-P2.15-LS4.7, F.Cu at (151.8, 107.6)
- added K61: A, Uinio:KEY-SMD_4P-L4.2-W3.4-P2.15-LS4.7, F.Cu at (160.4, 78.3)
- added K62: A, Uinio:KEY-SMD_4P-L4.2-W3.4-P2.15-LS4.7, F.Cu at (160.4, 88.0)
- added K63: A, Uinio:KEY-SMD_4P-L4.2-W3.4-P2.15-LS4.7, F.Cu at (160.4, 97.8)
- added K64: A, Uinio:KEY-SMD_4P-L4.2-W3.4-P2.15-LS4.7, F.Cu at (160.4, 107.6)
- added K7: A, Uinio:KEY-SMD_4P-L4.2-W3.4-P2.15-LS4.7, F.Cu at (126.0, 88.0)
- added K8: A, Uinio:KEY-SMD_4P-L4.2-W3.4-P2.15-LS4.7, F.Cu at (134.6, 88.0)
- added K9: A, Uinio:KEY-SMD_4P-L4.2-W3.4-P2.15-LS4.7, F.Cu at (108.8, 97.8)
- added R1: 10K, Resistor_SMD:R_0402_1005Metric, F.Cu at (132.0, 59.6)
- added R10: 10K, Resistor_SMD:R_0402_1005Metric, F.Cu at (163.2, 69.6)
- added R11: 10K, Resistor_SMD:R_0402_1005Metric, F.Cu at (166.1, 61.7)
- added R12: 10K, Resistor_SMD:R_0402_1005Metric, F.Cu at (166.1, 63.7)
- added R13: 10K, Resistor_SMD:R_0402_1005Metric, F.Cu at (166.1, 65.7)
- added R14: 10K, Resistor_SMD:R_0402_1005Metric, F.Cu at (166.1, 67.6)
- added R15: 2K, Resistor_SMD:R_0402_1005Metric, F.Cu at (135.2, 53.3)
- added R2: 10K, Resistor_SMD:R_0402_1005Metric, F.Cu at (132.0, 61.6)
- added R3: 10K, Resistor_SMD:R_0402_1005Metric, F.Cu at (132.0, 63.6)
- added R4: 10K, Resistor_SMD:R_0402_1005Metric, F.Cu at (132.0, 65.6)
- added R5: 10K, Resistor_SMD:R_0402_1005Metric, F.Cu at (132.0, 67.6)
- added R6: 10K, Resistor_SMD:R_0402_1005Metric, F.Cu at (163.2, 61.7)
- added R7: 10K, Resistor_SMD:R_0402_1005Metric, F.Cu at (163.2, 63.7)
- added R8: 10K, Resistor_SMD:R_0402_1005Metric, F.Cu at (163.2, 65.7)
- added R9: 10K, Resistor_SMD:R_0402_1005Metric, F.Cu at (163.2, 67.6)
- added U1: CH452A, Uinio:SOIC-28_L17.9-W7.5-P1.27-LS10.3-BL, F.Cu at (147.4, 65.3)
- added U2: EC1106S, Uinio:SW-SMD_EC1106S, F.Cu at (114.4, 65.3)
- added U3: EC1106S, Uinio:SW-SMD_EC1106S, F.Cu at (180.7, 65.3)
Other:
- board outline added: 89.5 x 99.6 mm

Commit message: update
Parts:
- moved R13 39.8 mm to (126.6, 61.0)
- moved C2 39.3 mm to (168.2, 65.9), turned to 180 degrees
- moved C4 39.3 mm to (168.2, 61.6), turned to 180 degrees
- moved C6 39.1 mm to (168.2, 69.8), turned to 180 degrees
- moved R10 36.9 mm to (126.6, 65.7)
- moved R9 36.8 mm to (126.6, 70.9)
- moved C7 27.6 mm to (152.5, 56.9), turned to 180 degrees
- moved R1 26.9 mm to (154.9, 73.6), turned to -90 degrees
- moved R2 24.1 mm to (152.9, 73.6), turned to -90 degrees
- moved R8 23.7 mm to (140.9, 73.6), turned to -90 degrees
- moved R7 22.6 mm to (142.9, 73.6), turned to -90 degrees
- moved R6 21.9 mm to (144.9, 73.6), turned to -90 degrees
- moved R3 21.4 mm to (150.9, 73.6), turned to -90 degrees
- moved R4 18.7 mm to (148.9, 73.6), turned to -90 degrees
- moved R5 16.1 mm to (146.9, 73.6), turned to -90 degrees
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Other:
- board size 89.5 x 99.6 mm -> 89.5 x 99.1 mm

Commit message: PCB Layout.
Parts:
- added SW2: RKJXV1224005, Uinio:SW-TH_RKJXV1224005, F.Cu at (178.7, 61.8)
- moved D1 51.0 mm to (189.7, 77.4), turned to -90 degrees
- moved J2 50.5 mm to (125.1, 53.0)
- moved R15 49.7 mm to (189.7, 80.6), turned to 180 degrees
- moved C7 45.3 mm to (189.6, 82.9)
- moved U3 40.5 mm to (140.1, 63.9), turned to 90 degrees
- moved U1 33.9 mm to (178.4, 79.4)
- moved R1 33.6 mm to (185.6, 87.3)
- moved R2 33.6 mm to (183.6, 87.3)
- moved R3 33.6 mm to (181.6, 87.3)
- moved R4 33.6 mm to (179.6, 87.3)
- moved R5 33.6 mm to (177.6, 87.3)
- moved R6 33.6 mm to (175.6, 87.3)
- moved R7 33.6 mm to (173.6, 87.3)
- moved R8 33.6 mm to (171.6, 87.3)
- moved R14 21.4 mm to (151.4, 57.6), turned to 0 degrees
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Other:
- board size 89.5 x 99.1 mm -> 93.3 x 99.1 mm
- board text added: "#"
- board text added: "$"
- board text added: "%"
- board text added: "&"
- board text added: "("
- board text added: ")"
- board text added: "*"
- board text added: "+"
- board text added: "-"
- board text added: "."
- board text added: "0"
- board text added: "1"
- board text added: "2"
- board text added: "3"
- board text added: "4"
- board text added: "5"
- board text added: "6"
- board text added: "7"
- board text added: "8"
- board text added: "9"
- board text added: "="
- board text added: "@"
- board text added: "A"
- board text added: "ALT"
- board text added: "B"
- board text added: "C"
- board text added: "CTRL"
- board text added: "D"
- board text added: "E"
- board text added: "ENTER"
- board text added: "F"
- board text added: "G"
- board text added: "H"
- board text added: "I"
- board text added: "J"
- board text added: "K"
- board text added: "L"
- board text added: "M"
- board text added: "N"
- board text added: "O"
- board text added: "P"
- board text added: "Q"
- board text added: "R"
- board text added: "S"
- board text added: "SHIFT"
- board text added: "SPACE"
- board text added: "T"
- board text added: "U"
- board text added: "UINIO-Keyboard"
- board text added: "UinIO.com"
- board text added: "V"
- board text added: "Version 1.0.0"
- board text added: "W"
- board text added: "X"
- board text added: "Y"
- board text added: "Z"
- board text added: "^"
- board text added: "×"
- board text added: "÷"
- board text added: "！"

Commit message: Update PCB Layout.
Parts:
- added C10: 0.01uF, Capacitor_SMD:C_0402_1005Metric, F.Cu at (163.4, 60.8)
- added C8: 0.01uF, Capacitor_SMD:C_0402_1005Metric, F.Cu at (163.4, 69.2)
- added C9: 0.01uF, Capacitor_SMD:C_0402_1005Metric, F.Cu at (163.4, 64.4)
- added D2: LED_Red, LED_SMD:LED_0603_1608Metric, F.Cu at (118.0, 57.1)
- added D3: LED_Red, LED_SMD:LED_0603_1608Metric, F.Cu at (139.2, 57.1)
- added D4: LED_Red, LED_SMD:LED_0603_1608Metric, F.Cu at (160.5, 57.1)
- added D5: LED_Red, LED_SMD:LED_0603_1608Metric, F.Cu at (188.7, 56.1)
- added J4: Conn_01x05_Pin, Connector_PinHeader_2.54mm:PinHeader_1x05_P2.54mm_Vertical, F.Cu at (177.5, 52.1)
- added J5: Conn_01x05_Pin, Connector_PinHeader_2.54mm:PinHeader_1x05_P2.54mm_Vertical, F.Cu at (140.8, 52.1)
- added R16: 2K, Resistor_SMD:R_0402_1005Metric, F.Cu at (120.9, 57.4)
- added R17: 2K, Resistor_SMD:R_0402_1005Metric, F.Cu at (142.1, 57.4)
- added R18: 2K, Resistor_SMD:R_0402_1005Metric, F.Cu at (163.4, 57.4)
- added R19: 10K, Resistor_SMD:R_0402_1005Metric, F.Cu at (163.4, 65.6)
- added R20: 10K, Resistor_SMD:R_0402_1005Metric, F.Cu at (163.4, 70.3)
- added R21: 10K, Resistor_SMD:R_0402_1005Metric, F.Cu at (163.4, 59.7)
- added R22: 2K, Resistor_SMD:R_0402_1005Metric, F.Cu at (189.3, 58.2)
- added SW1: SWITCH_SS12D00G3, Uinio:SW-TH_SS-12D01-GX, F.Cu at (168.3, 79.3)
- added U4: EC1106S, Uinio:SW-SMD_EC1106S, F.Cu at (152.6, 64.1)
- moved R14 9.81 mm to (142.1, 60.8)
- moved R11 9.58 mm to (142.1, 65.5)
- moved R12 9.48 mm to (142.1, 70.3)
- moved C6 9.31 mm to (142.1, 59.7)
- moved C4 9.28 mm to (142.1, 64.4)
- moved C2 9.26 mm to (142.1, 69.1)
- moved U3 8.66 mm to (131.5, 64.1)
- moved C5 4.06 mm to (120.9, 59.7)
- moved R13 4.06 mm to (120.9, 60.8)
- moved R9 3.98 mm to (120.9, 65.5)
- moved C3 3.98 mm to (120.9, 64.4)
- moved C1 3.62 mm to (120.9, 69.1)
- moved R10 3.62 mm to (120.9, 70.3)
- moved U2 2.94 mm to (110.3, 64.1)
- moved SW2 2.44 mm to (180.7, 63.2)
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Connections:
- SW2 pad 1: unconnected-(SW2-B-Pad1) -> /Rocker_VCC
- SW2 pad 10: unconnected-(SW2-GND-Pad10) -> Net-(SW2-GND-Pad10)
- SW2 pad 2: unconnected-(SW2-DTA-Pad2) -> /Rocker_Y
- SW2 pad 3: unconnected-(SW2-A-Pad3) -> /Rocker_GND
- SW2 pad 4: unconnected-(SW2-A-Pad4) -> /Rocker_VCC
- SW2 pad 5: unconnected-(SW2-DTA-Pad5) -> /Rocker_X
- SW2 pad 6: unconnected-(SW2-B-Pad6) -> /Rocker_GND
- SW2 pad 7: unconnected-(SW2-GND-Pad7) -> Net-(SW2-GND-Pad7)
- SW2 pad 8: unconnected-(SW2-GND-Pad8) -> Net-(SW2-GND-Pad7)
- SW2 pad 9: unconnected-(SW2-GND-Pad9) -> Net-(SW2-GND-Pad10)
- SW2 pad a: Net-(SW2-Pada) -> /Rocker_GND
- SW2 pad b: Net-(SW2-Pada) -> /Rocker_SW
- SW2 pad c: Net-(SW2-Padc) -> /Rocker_GND
- SW2 pad d: Net-(SW2-Padc) -> /Rocker_SW
Other:
- board size 93.3 x 99.1 mm -> 100 x 100 mm
- board text added: "/"
- board text added: "<"
- board text added: ">"
- board text added: "BACK"
- board text added: "DEL"
- board text added: "ESC"
- board text added: "GND"
- board text added: "SW"
- board text added: "VCC"
- board text added: "\"
- board text added: "test"
- board text added: "{"
- board text added: "|"
- board text added: "}"
- board text added: "~"
- board text added: "。"
- board text added: "《"
- board text added: "》"
- board text added: "，"
- board text added: "："
- board text added: "；"
- board text added: "？"
- board text removed: "÷"

Commit message: update
Parts:
- added ?: LOGO, LOGO, B.Cu at (146.9, 101.6)
- moved J3 17.3 mm to (123.8, 52.1)
- moved J2 17.1 mm to (106.5, 52.1)
- moved D5 1.17 mm to (189.7, 56.7)
- moved SW2 1.11 mm to (181.8, 63.4)
- moved J4 0.64 mm to (178.2, 52.1)
- moved J1 0.48 mm to (158.4, 52.1)
- moved R22 0.41 mm to (189.6, 58.4), turned to 180 degrees
- moved J5 0.32 mm to (141.1, 52.1)
Connections:
- C7 pad 1: /LOAD -> /VCC
- J1 pad 3: /LOAD -> /VCC
- J4 pad 1: /Rocker_GND -> /Rocker_SW
- J4 pad 2: /Rocker_VCC -> /Rocker_X
- J4 pad 3: /Rocker_X -> /Rocker_Y
- J4 pad 4: /Rocker_Y -> /Rocker_VCC
- J4 pad 5: /Rocker_SW -> /Rocker_GND
- R15 pad 2: /LOAD -> /VCC
- R22 pad 2: /Rocker_GND -> /Rocker_SW
- SW1 pad 1: unconnected-(SW1-Pad1) -> GND
- SW1 pad 2: unconnected-(SW1-Pad2) -> /LOAD
- SW1 pad 3: unconnected-(SW1-Pad3) -> /VCC
- U1 pad 23: /LOAD -> /VCC
Other:
- board text added: "键 盘 I²C 地 址 选 择"

Commit message: Update PCB.
Parts:
- moved D5 0.14 mm to (189.6, 56.6), turned to 180 degrees
- moved R22 0.14 mm to (189.5, 58.3), turned to 0 degrees
Other:
- outline, holes or cut-outs redrawn
Changed lines of the file:
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@@
   )
   (footprint "LED_SMD:LED_0603_1608Metric" (layer "F.Cu")
-    (at 189.7175 56.7)
+    (at 189.61 56.61 180)
     (descr "LED SMD 0603 (1608 Metric), square (rectangular) end terminal, IPC_7351 nominal, (Body size source: http://www.tortai-tech.com/upload/download/2011102023233369053.pdf), generated with kicad-footprint-generator")
     (tags "LED")
@@
     (property "ki_keywords" "LED diode")
     (attr smd)
-    (fp_text reference "D5" (at 2.1975 0.06) (layer "F.SilkS")
+    (fp_text reference "D5" (at 1.89 -0.01 90) (layer "F.SilkS")
         (effects (font (size 0.7 0.7) (thickness 0.1)))
     )
@@
     (fp_line (start 0.8 0.4) (end 0.8 -0.4)
       (stroke (width 0.1) (type solid)) (layer "F.Fab"))
-    (pad "1" smd roundrect (at -0.7875 0) (size 0.875 0.95) (layers "F.Cu" "F.Paste" "F.Mask") (roundrect_rratio 0.25)
+    (pad "1" smd roundrect (at -0.7875 0 180) (size 0.875 0.95) (layers "F.Cu" "F.Paste" "F.Mask") (roundrect_rratio 0.25)
       (net 57 "/Rocker_GND") (pinfunction "K") (pintype "passive"))
-    (pad "2" smd roundrect (at 0.7875 0) (size 0.875 0.95) (layers "F.Cu" "F.Paste" "F.Mask") (roundrect_rratio 0.25)
+    (pad "2" smd roundrect (at 0.7875 0 180) (size 0.875 0.95) (layers "F.Cu" "F.Paste" "F.Mask") (roundrect_rratio 0.25)
       (net 59 "Net-(D5-A)") (pinfunction "A") (pintype "passive"))
     (model "${KICAD6_3DMODEL_DIR}/LED_SMD.3dshapes/LED_0603_1608Metric.wrl"
@@
   )
   (footprint "Resistor_SMD:R_0402_1005Metric" (layer "F.Cu")
-    (at 189.6275 58.4 180)
+    (at 189.52 58.31)
     (descr "Resistor SMD 0402 (1005 Metric), square (rectangular) end terminal, IPC_7351 nominal, (Body size source: IPC-SM-782 page 72, https://www.pcb-3d.com/wordpress/wp-content/uploads/ipc-sm-782a_amendment_1_and_2.pdf), generated with kicad-footprint-generator")
     (tags "resistor")
@@
     (property "ki_keywords" "R res resistor")
     (attr smd)
-    (fp_text reference "R22" (at -2 -0.04) (layer "F.SilkS")
+    (fp_text reference "R22" (at 0.0025 0.99) (layer "F.SilkS")
         (effects (font (size 0.7 0.7) (thickness 0.1)))
     )
@@
     (fp_line (start 0.525 0.27) (end -0.525 0.27)
       (stroke (width 0.1) (type solid)) (layer "F.Fab"))
-    (pad "1" smd roundrect (at -0.51 0 180) (size 0.54 0.64) (layers "F.Cu" "F.Paste" "F.Mask") (roundrect_rratio 0.25)
+    (pad "1" smd roundrect (at -0.51 0) (size 0.54 0.64) (layers "F.Cu" "F.Paste" "F.Mask") (roundrect_rratio 0.25)
       (net 59 "Net-(D5-A)") (pintype "passive"))
-    (pad "2" smd roundrect (at 0.51 0 180) (size 0.54 0.64) (layers "F.Cu" "F.Paste" "F.Mask") (roundrect_rratio 0.25)
+    (pad "2" smd roundrect (at 0.51 0) (size 0.54 0.64) (layers "F.Cu" "F.Paste" "F.Mask") (roundrect_rratio 0.25)
       (net 51 "/Rocker_SW") (pintype "passive"))
     (model "${KICAD6_3DMODEL_DIR}/Resistor_SMD.3dshapes/R_0402_1005Metric.wrl"
@@
     (stroke (width 0.1) (type default)) (layer "F.SilkS"))
   (gr_line (start 102.445 50.8) (end 192.445 50.8)
-    (stroke (width 0.1) (type default)) (layer "Edge.Cuts"))
-  (gr_arc (start 97.445 55.8) (mid 98.909466 52.264466) (end 102.445 50.8)
-    (stroke (width 0.1) (type default)) (layer "Edge.Cuts"))
+    (stroke (width 0.1) (type default)) (layer "Dwgs.User"))
+  (gr_arc (start 97.445 55.8) (mid 98.909466 52.264467) (end 102.445 50.8)
+    (stroke (width 0.1) (type default)) (layer "Dwgs.User"))
   (gr_line (start 192.445 150.8) (end 102.445 150.8)
-    (stroke (width 0.1) (type default)) (layer "Edge.Cuts"))
+    (stroke (width 0.1) (type default)) (layer "Dwgs.User"))
   (gr_line (start 97.445 145.8) (end 97.445 55.8)
-    (stroke (width 0.1) (type default)) (layer "Edge.Cuts"))
+    (stroke (width 0.1) (type default)) (layer "Dwgs.User"))
   (gr_line (start 197.445 55.8) (end 197.445 145.8)
-    (stroke (width 0.1) (type default)) (layer "Edge.Cuts"))
-  (gr_arc (start 197.445 145.8) (mid 195.980534 149.335534) (end 192.445 150.8)
-    (stroke (width 0.1) (type default)) (layer "Edge.Cuts"))
-  (gr_arc (start 192.445 50.8) (mid 195.980534 52.264466) (end 197.445 55.8)
-    (stroke (width 0.1) (type default)) (layer "Edge.Cuts"))
-  (gr_arc (start 102.445 150.8) (mid 98.909466 149.335534) (end 97.445 145.8)
-    (stroke (width 0.1) (type default)) (layer "Edge.Cuts"))
+    (stroke (width 0.1) (type default)) (layer "Dwgs.User"))
+  (gr_arc (start 197.445 145.8) (mid 195.980534 149.335533) (end 192.445 150.8)
+    (stroke (width 0.1) (type default)) (layer "Dwgs.User"))
+  (gr_arc (start 192.445 50.8) (mid 195.980533 52.264466) (end 197.445 55.8)
+    (stroke (width 0.1) (type default)) (layer "Dwgs.User"))
+  (gr_arc (start 102.445 150.8) (mid 98.909467 149.335534) (end 97.445 145.8)
+    (stroke (width 0.1) (type default)) (layer "Dwgs.User"))
+  (gr_line (start 197.42 55.8) (end 197.42 145.8)
+    (stroke (width 0.1) (type solid)) (layer "Edge.Cuts"))
+  (gr_circle (center 193.42 100.8) (end 195.02 100.8)
+    (stroke (width 0.1) (type solid)) (fill none) (layer "Edge.Cuts"))
+  (gr_circle (center 193.42 54.8) (end 195.02 54.8)
+    (stroke (width 0.1) (type solid)) (fill none) (layer "Edge.Cuts"))
+  (gr_line (start 97.42 145.8) (end 97.42 55.8)
+    (stroke (width 0.1) (type solid)) (layer "Edge.Cuts"))
+  (gr_circle (center 101.42 100.8) (end 103.02 100.8)
+    (stroke (width 0.1) (type solid)) (fill none) (layer "Edge.Cuts"))
+  (gr_line (start 192.42 150.8) (end 102.42 150.8)
+    (stroke (width 0.1) (type solid)) (layer "Edge.Cuts"))
+  (gr_line (start 102.42 50.8) (end 192.42 50.8)
+    (stroke (width 0.1) (type solid)) (layer "Edge.Cuts"))
+  (gr_circle (center 101.42 146.8) (end 103.02 146.8)
+    (stroke (width 0.1) (type solid)) (fill none) (layer "Edge.Cuts"))
+  (gr_circle (center 193.42 146.8) (end 195.02 146.8)
+    (stroke (width 0.1) (type solid)) (fill none) (layer "Edge.Cuts"))
+  (gr_arc (start 197.42 145.8) (mid 195.955534 149.335534) (end 192.42 150.8)
+    (stroke (width 0.1) (type solid)) (layer "Edge.Cuts"))
+  (gr_arc (start 97.42 55.8) (mid 98.884466 52.264466) (end 102.42 50.8)
+    (stroke (width 0.1) (type solid)) (layer "Edge.Cuts"))
+  (gr_arc (start 192.42 50.8) (mid 195.955534 52.264466) (end 197.42 55.8)
+    (stroke (width 0.1) (type solid)) (layer "Edge.Cuts"))
+  (gr_arc (start 102.42 150.8) (mid 98.884466 149.335534) (end 97.42 145.8)
+    (stroke (width 0.1) (type solid)) (layer "Edge.Cuts"))
+  (gr_circle (center 101.42 54.8) (end 103.02 54.8)
+    (stroke (width 0.1) (type solid)) (fill none) (layer "Edge.Cuts"))
   (gr_rect (start 176.98 119.4) (end 178.5 119.86)
     (stroke (width 0.15) (type default)) (fill none) (layer "User.5"))
@@
     )
   )
+  (group "" (id ceb1d74c-8739-4aca-b8fc-6dd2289b4764)
+    (members
+      0a4962ac-2328-47da-a5e1-3e486024eaf7
+      2c6b0e59-15f4-4a6c-89f7-c2f41cdd9f03
+      57eae83e-f587-441e-b203-20e67aa666df
+      5aff40e4-02d7-483a-8b6c-abb36c0bcd4a
+      661b7036-4107-4c22-8c2d-5f9140fd50ea
+      8d60a7ff-e090-428a-acc6-b29956cf12b4
+      911eba2f-35b1-46ba-b5ba-0b494d2823db
+      ac427ab5-93cb-4669-91b0-73e3ee4a8ac5
+      bb18781c-28cb-4036-b177-95f4fcf31aa6
+      bdbaeb25-2017-4583-a8f5-73ed6998d10d
+      bf6e69e5-8e0f-40e9-9e56-ed86aa895f6d
+      d44d7b95-8c11-4c16-85db-34fab31c8e19
+      e1585ae8-5fec-4912-8419-8cf8c55fc7da
+      e7231257-8f66-4946-a428-9562525d95ee
+    )
+  )

Commit message: Update PCB.
Parts:
- moved D5 0.21 mm to (189.6, 56.8)
Other:
- outline, holes or cut-outs redrawn
- board text added: "8×8 键 盘 I²C 地 址 选 择"
- board text added: "8×8 键盘"
- board text added: "碳膜摇杆"
- board text added: "编码器 A"
- board text added: "编码器 B"
- board text added: "编码器 C"
- board text added: "编码器A"
- board text added: "编码器B"
- board text added: "编码器C"
- board text removed: "键 盘 I²C 地 址 选 择"

Commit message: Complete PCB layout.
Parts:
- added G***: LOGO, LOGO, B.Cu at (147.2, 120.3)
- moved ? 10.5 mm to (147.1, 91.1)
Connections:
- J1 pad 1: /RST# -> /DCLK
- J1 pad 2: /DOUT -> GND
- J1 pad 3: /VCC -> /DOUT
- J1 pad 4: GND -> /RST#
- J1 pad 6: /DCLK -> /VCC
Other:
- board text added: "8×8"
- board text added: "INT"
- board text added: "RST"
- board text added: "SCL"
- board text added: "SDA"
- board text added: "扫描访问 UinIO.com"
- board text added: "键 盘 I²C 地 址 选 择"
- board text removed: "8×8 键 盘 I²C 地 址 选 择"
- board text removed: "test"
