File: UINIO-Keyboard.kicad_pcb (KiCad board)
At the start: 2 copper layers, 100 x 100 mm, 114 parts, among them J1 Conn_01x06_Pin, J2 Conn_01x05_Pin, J3 Conn_01x05_Pin, J4 Conn_01x05_Pin, J5 Conn_01x05_Pin, K1 A, K10 A, K11 A, K12 A, K13 A, K14 A, K15 A, K16 A, K17 A, K18 A, K19 A, K2 A, K20 A, K21 A, K22 A, K23 A, K24 A, K25 A, K26 A, K27 A, K28 A, K29 A, K3 A, K30 A, K31 A, K32 A, K33 A, K34 A, K35 A, K36 A, K37 A, K38 A, K39 A, K4 A, K40 A, K41 A, K42 A, K43 A, K44 A, K45 A, K46 A, K47 A, K48 A, K49 A, K5 A, K50 A, K51 A, K52 A, K53 A, K54 A, K55 A, K56 A, K57 A, K58 A, K59 A, K6 A, K60 A, K61 A, K62 A, K63 A, K64 A, K7 A, K8 A, K9 A, SW1 SWITCH_SS12D00G3, SW2 RKJXV1224005, U1 CH452A, U2 EC1106S, U3 EC1106S, U4 EC1106S

Commit message: Update PCB.
Connections:
- net /EC11-E-1 renamed /EC11-D-1
- net /EC11-E-2 renamed /EC11-D-2
- net /EC11-E-3 renamed /EC11-D-3
- J1 pad 2: GND -> /DIN
- J1 pad 4: /RST# -> /RST
- U1 pad 12: unconnected-(U1-RST-Pad12) -> /RST
- U1 pad 13: /RST# -> unconnected-(U1-RST#-Pad13)
- U1 pad 26: GND -> /DIN
Other:
- board text added: "'"
- board text added: "_"
- board text added: "`"
- board text added: "{dblquote}"

Commit message: Update PCB.
Parts:
- C3, C4, C9: value 0.01uF -> 0.1uF
- moved D3 21.3 mm to (117.9, 57.1)
- moved R16 21.2 mm to (142.1, 57.4)
- moved R17 21.2 mm to (121.0, 57.4)
- moved D2 21.1 mm to (139.1, 57.1)
- moved C1 4.75 mm to (120.9, 64.4)
- moved C3 4.75 mm to (120.9, 69.1)
- moved C2 4.75 mm to (142.1, 64.4)
- moved C4 4.75 mm to (142.1, 69.1)
- moved C8 4.75 mm to (163.4, 64.4)
- moved C9 4.75 mm to (163.4, 69.2)
- moved R10 4.74 mm to (120.9, 65.5)
- moved R9 4.74 mm to (120.9, 70.3)
- moved R19 4.74 mm to (163.4, 70.3)
- moved R20 4.74 mm to (163.4, 65.6)
- moved R11 4.74 mm to (142.1, 70.3)
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Connections:
- C1 pad 2: /EC11-GND-1 -> GND
- C10 pad 2: /EC11-GND-3 -> GND
- C2 pad 2: /EC11-GND-2 -> GND
- C3 pad 2: /EC11-GND-1 -> GND
- C4 pad 2: /EC11-GND-2 -> GND
- C5 pad 2: /EC11-GND-1 -> GND
- C6 pad 2: /EC11-GND-2 -> GND
- C8 pad 2: /EC11-GND-3 -> GND
- C9 pad 2: /EC11-GND-3 -> GND
- D2 pad 1: /EC11-GND-2 -> GND
- D3 pad 1: /EC11-GND-1 -> GND
- D4 pad 1: /EC11-GND-3 -> GND
- J2 pad 2: /EC11-GND-1 -> GND
- J2 pad 4: /EC11-B-1 -> /EC11-A-1
- J2 pad 5: /EC11-A-1 -> /EC11-B-1
- J3 pad 2: /EC11-GND-2 -> GND
- J3 pad 4: /EC11-B-2 -> /EC11-A-2
- J3 pad 5: /EC11-A-2 -> /EC11-B-2
- J4 pad 1: /Rocker_SW -> /Rocker_X
- J4 pad 2: /Rocker_X -> /Rocker_Y
- J4 pad 3: /Rocker_Y -> /Rocker_SW
- J4 pad 4: /Rocker_VCC -> /Rocker_GND
- J4 pad 5: /Rocker_GND -> /Rocker_VCC
- J5 pad 2: /EC11-GND-3 -> GND
- J5 pad 4: /EC11-B-3 -> /EC11-A-3
- J5 pad 5: /EC11-A-3 -> /EC11-B-3
- R22 pad 2: /Rocker_SW -> /Rocker_VCC
- U2 pad 2: /EC11-GND-1 -> GND
- U2 pad 4: /EC11-GND-1 -> GND
- U2 pad 6: /EC11-GND-1 -> GND
- U2 pad 7: /EC11-GND-1 -> GND
- U3 pad 2: /EC11-GND-2 -> GND
- U3 pad 4: /EC11-GND-2 -> GND
- U3 pad 6: /EC11-GND-2 -> GND
- U3 pad 7: /EC11-GND-2 -> GND
- U4 pad 2: /EC11-GND-3 -> GND
- U4 pad 4: /EC11-GND-3 -> GND
- U4 pad 6: /EC11-GND-3 -> GND
- U4 pad 7: /EC11-GND-3 -> GND
Routing:
- net Net-(K41-Pad1): track 0.00 -> 186.4 mm, vias 0 -> 7
- net /SEG4: track 0.00 -> 184.5 mm, vias 0 -> 8
- net /SEG0: track 0.00 -> 177.9 mm, vias 0 -> 8
- net /SEG5: track 0.00 -> 163.3 mm, vias 0 -> 10
- net /SEG6: track 0.00 -> 143.1 mm, vias 0 -> 5
- net /SEG2: track 0.00 -> 142.8 mm, vias 0 -> 5
- net /SEG3: track 0.00 -> 134.9 mm, vias 0 -> 7
- net /SEG1: track 0.00 -> 129.1 mm, vias 0 -> 7
- net Net-(K25-Pad1): track 0.00 -> 126.1 mm
- net Net-(K33-Pad1): track 0.00 -> 124.8 mm, vias 0 -> 2
- net /SEG7: track 0.00 -> 114.7 mm, vias 0 -> 5
- net Net-(K1-Pad1): track 0.00 -> 108.1 mm
- net Net-(K17-Pad1): track 0.00 -> 103.9 mm
- net Net-(K10-Pad1): track 0.00 -> 101.9 mm
- net Net-(K57-Pad1): track 0.00 -> 100.5 mm, vias 0 -> 3
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- added copper zone on B.Cu, net GND
- added copper zone on F.Cu, net GND

Commit message: Update PCB.
Parts:
- renumbered G*** to ?
Connections:
- D5 pad 1: /Rocker_GND -> GND
- J4 pad 4: /Rocker_GND -> GND
- SW2 pad 10: Net-(SW2-GND-Pad10) -> GND
- SW2 pad 3: /Rocker_GND -> GND
- SW2 pad 6: /Rocker_GND -> GND
- SW2 pad 7: Net-(SW2-GND-Pad7) -> GND
- SW2 pad 8: Net-(SW2-GND-Pad7) -> GND
- SW2 pad 9: Net-(SW2-GND-Pad10) -> GND
- SW2 pad a: /Rocker_GND -> GND
- SW2 pad c: /Rocker_GND -> GND
Routing:
- net /SEG3: track 134.9 -> 284.8 mm, vias 7 -> 13
- net /SEG1: track 129.1 -> 239.9 mm, vias 7 -> 11
- net /SEG2: track 142.8 -> 245.8 mm, vias 5 -> 9
- net Net-(K49-Pad1): track 48.2 -> 119.7 mm, vias 0 -> 7
- net /SEG7: track 114.7 -> 183.4 mm, vias 5 -> 8
- net /SEG0: track 177.9 -> 245.0 mm, vias 8 -> 12
- net /SEG6: track 143.1 -> 201.8 mm, vias 5 -> 7
- net GND: track 3.60 -> 42.2 mm, vias 0 -> 37
- net /VCC: track 46.7 -> 83.8 mm
- net /SEG5: track 163.3 -> 199.8 mm
- net /Rocker_VCC: track 15.7 -> 29.2 mm, vias 1 -> 2
- net /SEG4: track 184.5 -> 196.1 mm
- net Net-(SW2-GND-Pad10): track 10.0 -> 0.00 mm
- net Net-(K10-Pad1): track 101.9 -> 111.5 mm, vias 0 -> 2
- net Net-(K57-Pad1): track 100.5 -> 109.2 mm, vias 3 -> 5
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
Commit message: Update PCB.
Routing:
- net /SEG5: track 199.8 -> 243.6 mm, vias 10 -> 11
- net /SEG2: track 245.8 -> 268.4 mm
- net /SEG4: track 196.1 -> 218.4 mm, vias 8 -> 9
- net /SEG1: track 239.9 -> 257.9 mm
- net /SEG0: track 245.0 -> 262.3 mm, vias 12 -> 14
- net /SEG6: track 201.8 -> 216.7 mm
- net Net-(K49-Pad1): track 119.7 -> 133.2 mm, vias 7 -> 9
- net /SEG3: track 284.8 -> 287.6 mm
- net GND: track 42.2 -> 40.6 mm, vias 37 -> 47
- net /RST: track 44.4 -> 43.2 mm
- net /VCC: track 83.8 -> 84.9 mm
