File: UINIO-Keyboard.kicad_pcb (KiCad board)
At the start: 2 copper layers, 100 x 100 mm, 114 parts, among them J1 Conn_01x06_Pin, J2 Conn_01x05_Pin, J3 Conn_01x05_Pin, J4 Conn_01x05_Pin, J5 Conn_01x05_Pin, K1 A, K10 A, K11 A, K12 A, K13 A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

Commit message: Finish PCB layout.
Parts:
- moved ? 0.22 mm to (147.4, 120.3)
- moved ? 0.22 mm to (147.3, 91.1)
